File: hardware/TOS100-Shield_v16.sch (EAGLE design)
At the start: 63 parts, among them IC1 TMC260-PA, J1 POWER_JACKPTH, T1 N-Chn, T2 N-Chn, T3 P-Chn, T4 N-Chn

Commit message: updated layout and schematics
Other:
- moved on the sheet: DIR, EN, R10, R11, R12, R13, R14, R7, R8, R9, SG, STEP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
